Commit message: added obj_traj_est

File: src/simulator/urdf/april_tag.xacro (robot description, xacro)
@@ -1,5 +1,5 @@
 <?xml version ="1.0"?>
 <robot name="april_tag" xmlns:xacro="http://ros.org/wiki/xacro">
-	<link name="base_link">
+	<link name="april_tag_base_link">
 		<visual>
 			<geometry>
@@ -19,5 +19,5 @@
     </collision>
   </link>
-	<gazebo reference="base_link">
+	<gazebo reference="april_tag_base_link">
 		<material>Apriltag1</material>
   </gazebo>
@@ -28,5 +28,5 @@
         <odometryFrame>odom</odometryFrame>
         <odometryRate>10.0</odometryRate>
-        <robotBaseFrame>base_link</robotBaseFrame>
+        <robotBaseFrame>april_tag_link</robotBaseFrame>
       </plugin>
   </gazebo>

File: src/simulator/urdf/camera.xacro (robot description, xacro)
@@ -73,7 +73,7 @@
         <commandTopic>cmd_vel</commandTopic>
         <odometryTopic>odom</odometryTopic>
-        <odometryFrame>odom</odometryFrame>
+        <odometryFrame>drone_odom</odometryFrame>
         <odometryRate>10.0</odometryRate>
-        <robotBaseFrame>camera_link</robotBaseFrame>
+        <robotBaseFrame>drone_link</robotBaseFrame>
       </plugin>
   </gazebo>

Commit message: target trajectory estimation working

File: src/simulator/urdf/april_tag.xacro (robot description, xacro)
@@ -6,5 +6,5 @@
 				<box size="0.2 0.2 0.001"/>
 			</geometry>
-      <origin xyz="0.2 0 0" rpy="0 0 0"/>
+      <origin xyz="0 0 0" rpy="0 0 0"/>
 		</visual>
 		<inertial>
@@ -27,5 +27,5 @@
         <odometryTopic>odom</odometryTopic>
         <odometryFrame>odom</odometryFrame>
-        <odometryRate>10.0</odometryRate>
+        <odometryRate>20.0</odometryRate>
         <robotBaseFrame>april_tag_link</robotBaseFrame>
       </plugin>

File: src/simulator/urdf/camera.xacro (robot description, xacro)
@@ -7,5 +7,5 @@
 	<parent link="world"/>
 	<child link="camera_link"/>
-	<origin xyz="0.2 0 0.5" rpy="0.0 ${pi/2} ${pi/2}"/>
+	<origin xyz="0 0 3" rpy="0.0 ${pi/2} ${pi/2}"/>
 </joint>
 <link name="camera_link">
@@ -74,5 +74,5 @@
         <odometryTopic>odom</odometryTopic>
         <odometryFrame>drone_odom</odometryFrame>
-        <odometryRate>10.0</odometryRate>
+        <odometryRate>20.0</odometryRate>
         <robotBaseFrame>drone_link</robotBaseFrame>
       </plugin>

Commit message: Commented code

File: src/simulator/urdf/april_tag.xacro (robot description, xacro)
@@ -1,5 +1,8 @@
 <?xml version ="1.0"?>
 <robot name="april_tag" xmlns:xacro="http://ros.org/wiki/xacro">
-	<link name="april_tag_base_link">
+  <material name="white">
+    <color rgba="0.8 0.8 0.8 1"/>
+  </material>
+	<link name="april_tag_link">
 		<visual>
 			<geometry>
@@ -7,4 +10,5 @@
 			</geometry>
       <origin xyz="0 0 0" rpy="0 0 0"/>
+      <material name = "white"/>
 		</visual>
 		<inertial>
@@ -19,5 +23,5 @@
     </collision>
   </link>
-	<gazebo reference="april_tag_base_link">
+	<gazebo reference="april_tag_link">
 		<material>Apriltag1</material>
   </gazebo>
@@ -32,26 +36,2 @@
   </gazebo>
 </robot>
-<!-- <robot name="april_tag" xmlns:xacro="http://ros.org/wiki/xacro">
-  <link name="base_link">
-    <inertial>
-      <origin xyz="2 0 0" />
-      <mass value="1.0" />
-      <inertia  ixx="1.0" ixy="0.0"  ixz="0.0"  iyy="100.0"  iyz="0.0"  izz="1.0" />
-    </inertial>
-    <visual>
-      <origin xyz="2 0 1"/>
-      <geometry>
-        <box size="1 1 2" />
-      </geometry>
-    </visual>
-    <collision>
-      <origin xyz="2 0 1"/>
-      <geometry>
-        <box size="1 1 2" />
-      </geometry>
-    </collision>
-  </link>
-  <gazebo reference="base_link">
-    <material>Gazebo/Blue</material>
-  </gazebo>
-</robot> -->

File: src/simulator/urdf/camera.xacro (robot description, xacro)
@@ -1,37 +1,42 @@
-<?xml version ="1.0"?>
-<robot name="camera" xmlns:xacro="http://ros.org/wiki/xacro">
-<link name="world">
-	<origin xyz="0 0 0"/>
+<?xml version = "1.0"?>
+<robot name = "camera" xmlns:xacro = "http://ros.org/wiki/xacro">
+<xacro:arg name = "drone_height" default = "3" />
+<material name="red">
+  <color rgba="0.8 0 0 1"/>
+</material>
+<link name = "world">
+	<origin xyz = "0 0 0"/>
 </link>
-<joint name="camera_joint" type="floating">
-	<parent link="world"/>
-	<child link="camera_link"/>
-	<origin xyz="0 0 3" rpy="0.0 ${pi/2} ${pi/2}"/>
+<joint name = "camera_joint" type = "floating">
+	<parent link = "world"/>
+	<child link = "drone_link"/>
+	<origin xyz = "0 0 $(arg drone_height)" rpy = "0.0 ${pi / 2} ${pi / 2}"/>
 </joint>
-<link name="camera_link">
+<link name = "drone_link">
     <collision>
-      <origin xyz="0 0 0" rpy="0 0 0"/>
+      <origin xyz = "0 0 0" rpy = "0 0 0"/>
       <geometry>
-    <box size="0.01 0.01 0.01"/>
+    <box size="0.10 0.10 0.10"/>
       </geometry>
     </collision>
     <visual>
-      <origin xyz="0 0 0" rpy="0 0 0"/>
+      <origin xyz = "0 0 0" rpy = "0 0 0"/>
       <geometry>
-    <box size="0.01 0.01 0.01"/>
+    <box size = "0.10 0.10 0.10"/>
       </geometry>
-      <material name="red"/>
+      <material name = "red"/>
     </visual>
     <inertial>
-      <mass value="1e-5" />
-      <origin xyz="0 0 0" rpy="0 0 0"/>
-      <inertia ixx="1e-6" ixy="0" ixz="0" iyy="1e-6" iyz="0" izz="1e-6" />
+      <mass value = "1e-5" />
+      <origin xyz = "0 0 0" rpy = "0 0 0"/>
+      <inertia ixx = "1e-6" ixy = "0" ixz = "0" iyy = "1e-6" iyz = "0" izz = "1e-6" />
     </inertial>
   </link>
-  <gazebo reference="camera_link">
+  <gazebo reference = "drone_link">
+    <material>Gazebo/Red</material>
     <turnGravityOff>true</turnGravityOff>
-    <sensor type="camera" name="camera">
+    <sensor type = "camera" name = "camera">
       <update_rate>30.0</update_rate>
-      <camera name="head">
+      <camera name = "head">
         <horizontal_fov>1.3962634</horizontal_fov>
         <image>
@@ -53,5 +58,5 @@
         </noise>
       </camera>
-      <plugin name="camera_controller" filename="libgazebo_ros_camera.so">
+      <plugin name = "camera_controller" filename = "libgazebo_ros_camera.so">
         <alwaysOn>true</alwaysOn>
         <updateRate>0.0</updateRate>
@@ -59,5 +64,5 @@
         <imageTopicName>image_raw</imageTopicName>
         <cameraInfoTopicName>camera_info</cameraInfoTopicName>
-        <frameName>camera_link</frameName>
+        <frameName>drone_link</frameName>
         <hackBaseline>0.07</hackBaseline>
         <distortionK1>0.0</distortionK1>
@@ -70,5 +75,5 @@
   </gazebo>
   <gazebo>
-    <plugin name="drone_controller" filename="libgazebo_ros_planar_move.so">
+    <plugin name = "drone_controller" filename = "libgazebo_ros_planar_move.so">
         <commandTopic>cmd_vel</commandTopic>
         <odometryTopic>odom</odometryTopic>
@@ -78,6 +83,3 @@
       </plugin>
   </gazebo>
-<!-- <gazebo>
-    <static>true</static>
-</gazebo> -->
 </robot>
